File: PCBs/nes_snes_4_port/nes_snes_4_port.sch (EAGLE design)
At the start: 24 parts, among them J1 RJ45, J2 RJ45, U1 74245, U2 MC74VHC1GT125, U3 MC74VHC1GT125, U4 MC74VHC1GT125, U5 MC74VHC1GT125

Commit message: Lots of work on the 4 port PCB. Added some shielded RJ45s to the library.
Parts:
- removed J1, J2: RJ45, TASLink:RJ45
- added J5, J6, J7, J8: RJ45, TASLink:RJ45
- added J9: RJ45-S-4, TASLink:RJ45-S-4
- added JP13, JP15, JP16, JP17, JP18, JP19, JP20: (no value), SparkFun-Connectors:M04PTH
- added JP14, JP6: (no value), SparkFun-Connectors:M081X08
- added R11, R12: 3.6k, rcl:R-US_0207/2V
- added U10, U7, U8, U9: MC74VHC1GT125, TASLink:MC74VHC1GT125
- JP5: device SparkFun-Connectors:M06SIP -> SparkFun-Connectors:M081X08
Connections:
- net P1_CLOCK_LV renamed CP2_CLOCK_LV
- net P1_IODATA_LV renamed CP3_CLOCK_LV
- net P1_LATCH_LV renamed CP2_LATCH_LV
- net P2_CLOCK_LV renamed CP3_LATCH_LV
- net P2_IODATA_LV renamed CP4_LATCH_LV
- net P2_LATCH_LV renamed CP4_CLOCK_LV
- removed net CONSOLE+5V: J1.2, J2.2, R1.1, R2.1, R3.1, R4.1, R5.1, R6.1, U2G$2.VCC, U3G$2.VCC, U4G$2.VCC, U5G$2.VCC
- removed net P1_CLOCK: J1.8, JP5.1, R1.2, U1A.B6
- removed net P1_D0: J1.4, U2G$1.Y
- removed net P1_D0_LV: JP12.3, JP8.3, U2G$1.A
- removed net P1_D0_OE_LV: JP11.3, U2G$1.OE
- removed net P1_D1: J1.5, U3G$1.Y
- removed net P1_D1_LV: JP12.4, JP8.4, U3G$1.A
- removed net P1_D1_OE_LV: JP11.4, U3G$1.OE
- removed net P1_IODATA: J1.3, JP5.3, R5.2, U1A.B4
- removed net P1_LATCH: J1.6, JP5.2, R3.2, U1A.B5
- removed net P2_CLOCK: J2.8, JP5.4, R2.2, U1A.B3
- removed net P2_D0: J2.4, U4G$1.Y
- removed net P2_D0_OE_LV: JP11.1, U4G$1.OE
- removed net P2_D1: J2.5, U5G$1.Y
- removed net P2_D1_LV: JP12.2, JP8.2, U5G$1.A
- removed net P2_D1_OE_LV: JP11.2, U5G$1.OE
- removed net P2_DO_LV: JP12.1, JP8.1, U4G$1.A
- removed net P2_IODATA: J2.3, JP5.6, R6.2, U1A.B1
- removed net P2_LATCH: J2.6, JP5.5, R4.2, U1A.B2
- new net CP1_+5V: J9P1.2, R1.1, R3.1, U2G$2.VCC, U3G$2.VCC
- new net CP1_CLOCK: J9P1.8, JP6.8, R1.2, U1A.B8
- new net CP1_CLOCK_LV: JP4.4, U1A.A8
- new net CP1_D0: J9P1.4, U2G$1.Y
- new net CP1_D0_LV: JP14.3, JP5.3, U2G$1.A
- new net CP1_D0_OE_LV: JP14.4, JP5.4, U2G$1.OE
- new net CP1_D1: J9P1.5, U3G$1.Y
- new net CP1_D1_LV: JP14.1, JP5.1, U3G$1.A
- new net CP1_D1_OE_LV: JP14.2, JP5.2, U3G$1.OE
- new net CP1_IODATA: J9P1.3
- new net CP1_LATCH: J9P1.6, JP6.7, R3.2, U1A.B7
- new net CP1_LATCH_LV: JP7.4, U1A.A7
- new net CP2_+5V: J9P2.2, R2.1, R4.1, U4G$2.VCC, U5G$2.VCC
- new net CP2_CLOCK: J9P2.8, JP6.6, R2.2, U1A.B6
- new net CP2_D0: J9P2.4, U4G$1.Y
- new net CP2_D0_OE_LV: JP14.8, JP5.8, U4G$1.OE
- new net CP2_D1: J9P2.5, U5G$1.Y
- new net CP2_D1_LV: JP14.5, JP5.5, U5G$1.A
- new net CP2_D1_OE_LV: JP14.6, JP5.6, U5G$1.OE
- new net CP2_DO_LV: JP14.7, JP5.7, U4G$1.A
- new net CP2_IODATA: J9P2.3
- new net CP2_LATCH: J9P2.6, JP6.5, R4.2, U1A.B5
- new net CP3_+5V: J9P3.2, R11.1, R5.1, U7G$2.VCC, U9G$2.VCC
- new net CP3_CLOCK: J9P3.8, JP6.4, R5.2, U1A.B4
- new net CP3_D0: J9P3.4, U7G$1.Y
- new net CP3_D0_LV: JP15.2, JP8.2, U7G$1.A
- new net CP3_D0_OE_LV: JP15.1, JP8.1, U7G$1.OE
- new net CP3_D1: J9P3.5, U9G$1.Y
- new net CP3_D1_LV: JP15.4, JP8.4, U9G$1.A
- new net CP3_D1_OE_LV: JP15.3, JP8.3, U9G$1.OE
- new net CP3_IODATA: J9P3.3
- new net CP3_LATCH: J9P3.6, JP6.3, R11.2, U1A.B3
- new net CP4_+5V: J9P4.2, R12.1, R6.1, U10G$2.VCC, U8G$2.VCC
- new net CP4_CLOCK: J9P4.8, JP6.2, R6.2, U1A.B2
- new net CP4_D0: J9P4.4, U8G$1.Y
- new net CP4_D0_OE_LV: JP11.4, JP20.4, U8G$1.OE
- new net CP4_D1: J9P4.5, U10G$1.Y
- new net CP4_D1_LV: JP11.1, JP20.1, U10G$1.A
- new net CP4_D1_OE_LV: JP11.2, JP20.2, U10G$1.OE
- new net CP4_DO_LV: JP11.3, JP20.3, U8G$1.A
- new net CP4_IODATA: J9P4.3
- new net CP4_LATCH: J9P4.6, JP6.1, R12.2, U1A.B1
- new net VP1_CLOCK: J5.8, JP19.1
- new net VP1_D0: J5.4, JP19.4
- new net VP1_D1: J5.5, JP19.3
- new net VP1_D2: J5.3
- new net VP1_D3: J5.7
- new net VP1_LATCH: J5.6, JP19.2
- new net VP2_CLOCK: J6.8, JP17.1
- new net VP2_D0: J6.4, JP17.4
- new net VP2_D1: J6.5, JP17.3
- new net VP2_D2: J6.3
- new net VP2_D3: J6.7
- new net VP2_LATCH: J6.6, JP17.2
- new net VP3_CLOCK: J7.8, JP18.4
- new net VP3_D0: J7.4, JP18.1
- new net VP3_D1: J7.5, JP18.2
- new net VP3_D2: J7.3
- new net VP3_D3: J7.7
- new net VP3_LATCH: J7.6, JP18.3
- new net VP4_CLOCK: J8.8, JP16.4
- new net VP4_D0: J8.4, JP16.1
- new net VP4_D1: J8.5, JP16.2
- new net VP4_D2: J8.3
- new net VP4_D3: J8.7
- new net VP4_LATCH: J8.6, JP16.3
- net +3V3: now also J5.2, J6.2, J7.2, J8.2, JP12.3; no longer JP1.3
- net GND: now also J5.1, J6.1, J7.1, J8.1, J9P1.1, J9P2.1, J9P3.1, J9P4.1, J9SHLD.S1, J9SHLD.S2, J9SHLD.S3, J9SHLD.S4, JP12.1, JP13.1, U10G$2.GND, U7G$2.GND, U8G$2.GND, U9G$2.GND; no longer J1.1, J2.1, U1A.B7, U1A.B8
Other:
- moved on the sheet: JP1, JP11, JP12, JP8, R2, R3, R4, R5, R6, U3, U3G$2, U4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

Commit message: 4 port PCB: Cleaned up the schematic.
Parts:
- removed JP10, JP2, JP3: (no value), SparkFun-Connectors:M04PTH
- added JP21: M09, SparkFun-Connectors:M09
- JP9: device SparkFun-Connectors:M04PTH -> SparkFun-Connectors:M081X08
Connections:
- net CP1_CLOCK: now also JP21.9; no longer JP6.8
- net CP1_LATCH: now also JP21.8; no longer JP6.7
- net CP2_CLOCK: now also JP21.7; no longer JP6.6
- net CP2_LATCH: now also JP21.6; no longer JP6.5
- net CP3_CLOCK: now also JP21.5; no longer JP6.4
- net CP3_LATCH: now also JP21.4; no longer JP6.3
- net CP4_CLOCK: now also JP21.3; no longer JP6.2
- net CP4_LATCH: now also JP21.2; no longer JP6.1
- net DEBUG0: now also JP6.1, JP9.1; no longer JP2.4, JP9.4
- net DEBUG1: now also JP6.2, JP9.2; no longer JP2.3, JP9.3
- net DEBUG2: now also JP6.3, JP9.3; no longer JP2.2, JP9.2
- net DEBUG3: now also JP6.4, JP9.4; no longer JP2.1, JP9.1
- net DEBUG4: now also JP6.5, JP9.5; no longer JP10.4, JP3.4
- net DEBUG5: now also JP6.6, JP9.6; no longer JP10.3, JP3.3
- net DEBUG6: now also JP6.7, JP9.7; no longer JP10.2, JP3.2
- net DEBUG7: now also JP6.8, JP9.8; no longer JP10.1, JP3.1
- net GND: now also JP21.1
Other:
- moved on the sheet: J5, J6, J7, J8, J9P1, J9P2, J9P3, J9P4, J9SHLD, JP1, JP11, JP12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
