File: PCBs/nes_visualization/nes_visualization.sch (EAGLE design)
At the start: 12 parts, among them U1 TLC59282

Commit message: NES Visualization: Changed the reference resistor to 0805 size.
Parts:
- R13: device rcl:R-US_R0603 -> rcl:R-US_R0805
Changed lines of the file:
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@@
 <attribute name="MOUSER#" value="80-C0603C104K5R"/>
 </part>
-<part name="R13" library="rcl" deviceset="R-US_" device="R0603" value="25k"/>
+<part name="R13" library="rcl" deviceset="R-US_" device="R0805" value="25k"/>
 <part name="GND16" library="supply1" deviceset="GND" device=""/>
 <part name="GND1" library="supply1" deviceset="GND" device=""/>
