File: PCBs/n64_4_port/n64_4_port.sch (EAGLE design)
At the start: 45 parts, among them J5 RJ45, J6 RJ45, J7 RJ45, J8 RJ45, J9 RJ45-S-4, U1 74245, U10 MC74VHC1GT125, U2 MC74VHC1GT125, U3 MC74VHC1GT125, U4 MC74VHC1GT125, U5 MC74VHC1GT125, U7 MC74VHC1GT125, U8 MC74VHC1GT125, U9 MC74VHC1GT125

Commit message: N64 pcb: Schematic complete and board routed.
Parts:
- removed J5, J6, J7, J8: RJ45, TASLink:RJ45
- removed JP15, JP16, JP17, JP18, JP19, JP20: (no value), SparkFun-Connectors:M04PTH
- removed JP21: M09, SparkFun-Connectors:M09
- removed JP9: (no value), SparkFun-Connectors:M081X08
- removed R1, R11, R12, R2, R3, R4, R5, R6: 3.6k, rcl:R-US_0207/2V
- removed U10, U3, U5, U9: MC74VHC1GT125, TASLink:MC74VHC1GT125
- added JP10, JP3: (no value), SparkFun-Connectors:M04PTH
- added JP2: (no value), SparkFun-Connectors:M05PTH
- JP1: value (none) -> M02PTH; device SparkFun-Connectors:M04PTH -> SparkFun-Connectors:M02PTH
- JP14, JP5, JP6: device SparkFun-Connectors:M081X08 -> SparkFun-Connectors:M04PTH
Connections:
- removed net CP1_+5V: C2.1, J9P1.2, R1.1, R3.1, U2G$2.VCC, U3G$2.VCC
- removed net CP1_CLOCK: J9P1.8, JP21.9, R1.2, U1A.B8
- removed net CP1_CLOCK_LV: JP4.4, U1A.A8
- removed net CP1_D0: J9P1.4, U2G$1.Y
- removed net CP1_D0_LV: JP14.3, JP5.3, U2G$1.A
- removed net CP1_D0_OE_LV: JP14.4, JP5.4, U2G$1.OE
- removed net CP1_D1: J9P1.5, U3G$1.Y
- removed net CP1_D1_LV: JP14.1, JP5.1, U3G$1.A
- removed net CP1_D1_OE_LV: JP14.2, JP5.2, U3G$1.OE
- removed net CP1_IODATA: J9P1.3
- removed net CP1_LATCH: J9P1.6, JP21.8, R3.2, U1A.B7
- removed net CP1_LATCH_LV: JP7.4, U1A.A7
- removed net CP2_+5V: C3.1, J9P2.2, R2.1, R4.1, U4G$2.VCC, U5G$2.VCC
- removed net CP2_CLOCK: J9P2.8, JP21.7, R2.2, U1A.B6
- removed net CP2_CLOCK_LV: JP4.3, U1A.A6
- removed net CP2_D0: J9P2.4, U4G$1.Y
- removed net CP2_D0_OE_LV: JP14.8, JP5.8, U4G$1.OE
- removed net CP2_D1: J9P2.5, U5G$1.Y
- removed net CP2_D1_LV: JP14.5, JP5.5, U5G$1.A
- removed net CP2_D1_OE_LV: JP14.6, JP5.6, U5G$1.OE
- removed net CP2_DO_LV: JP14.7, JP5.7, U4G$1.A
- removed net CP2_IODATA: J9P2.3
- removed net CP2_LATCH: J9P2.6, JP21.6, R4.2, U1A.B5
- removed net CP2_LATCH_LV: JP7.3, U1A.A5
- removed net CP3_+5V: C4.1, J9P3.2, R11.1, R5.1, U7G$2.VCC, U9G$2.VCC
- removed net CP3_CLOCK: J9P3.8, JP21.5, R5.2, U1A.B4
- removed net CP3_CLOCK_LV: JP4.2, U1A.A4
- removed net CP3_D0: J9P3.4, U7G$1.Y
- removed net CP3_D0_LV: JP15.2, JP8.2, U7G$1.A
- removed net CP3_D0_OE_LV: JP15.1, JP8.1, U7G$1.OE
- removed net CP3_D1: J9P3.5, U9G$1.Y
- removed net CP3_D1_LV: JP15.4, JP8.4, U9G$1.A
- removed net CP3_D1_OE_LV: JP15.3, JP8.3, U9G$1.OE
- removed net CP3_IODATA: J9P3.3
- removed net CP3_LATCH: J9P3.6, JP21.4, R11.2, U1A.B3
- removed net CP3_LATCH_LV: JP7.2, U1A.A3
- removed net CP4_+5V: C5.1, J9P4.2, R12.1, R6.1, U10G$2.VCC, U8G$2.VCC
- removed net CP4_CLOCK: J9P4.8, JP21.3, R6.2, U1A.B2
- removed net CP4_CLOCK_LV: JP4.1, U1A.A2
- removed net CP4_D0: J9P4.4, U8G$1.Y
- removed net CP4_D0_OE_LV: JP11.4, JP20.4, U8G$1.OE
- removed net CP4_D1: J9P4.5, U10G$1.Y
- removed net CP4_D1_LV: JP11.1, JP20.1, U10G$1.A
- removed net CP4_D1_OE_LV: JP11.2, JP20.2, U10G$1.OE
- removed net CP4_DO_LV: JP11.3, JP20.3, U8G$1.A
- removed net CP4_IODATA: J9P4.3
- removed net CP4_LATCH: J9P4.6, JP21.2, R12.2, U1A.B1
- removed net CP4_LATCH_LV: JP7.1, U1A.A1
- removed net VP1_CLOCK: J5.8, JP19.1
- removed net VP1_D0: J5.4, JP19.4
- removed net VP1_D1: J5.5, JP19.3
- removed net VP1_D2: J5.3
- removed net VP1_D3: J5.7
- removed net VP1_LATCH: J5.6, JP19.2
- removed net VP2_CLOCK: J6.8, JP17.1
- removed net VP2_D0: J6.4, JP17.4
- removed net VP2_D1: J6.5, JP17.3
- removed net VP2_D2: J6.3
- removed net VP2_D3: J6.7
- removed net VP2_LATCH: J6.6, JP17.2
- removed net VP3_CLOCK: J7.8, JP18.4
- removed net VP3_D0: J7.4, JP18.1
- removed net VP3_D1: J7.5, JP18.2
- removed net VP3_D2: J7.3
- removed net VP3_D3: J7.7
- removed net VP3_LATCH: J7.6, JP18.3
- removed net VP4_CLOCK: J8.8, JP16.4
- removed net VP4_D0: J8.4, JP16.1
- removed net VP4_D1: J8.5, JP16.2
- removed net VP4_D2: J8.3
- removed net VP4_D3: J8.7
- removed net VP4_LATCH: J8.6, JP16.3
- new net CP1_+3V3: C2.1, J9P1.2, U2G$2.VCC
- new net CP1_DATA: J9P1.3, JP2.5, U1A.B4, U2G$1.Y
- new net CP1_DATA_IN_LV: JP3.4, U1A.A4
- new net CP1_DATA_OUT_LV: JP4.1, JP7.1, U2G$1.A
- new net CP1_DATA_OUT_OE_LV: JP4.2, JP7.2, U2G$1.OE
- new net CP2_+3V3: C3.1, J9P2.2, U4G$2.VCC
- new net CP2_DATA: J9P2.3, JP2.4, U1A.B3, U4G$1.Y
- new net CP2_DATA_IN_LV: JP3.3, U1A.A3
- new net CP2_DATA_OUT_LV: JP4.3, JP7.3, U4G$1.A
- new net CP2_DATA_OUT_OE_LV: JP4.4, JP7.4, U4G$1.OE
- new net CP3_+3V3: C4.1, J9P3.2, U7G$2.VCC
- new net CP3_DATA: J9P3.3, JP2.3, U1A.B2, U7G$1.Y
- new net CP3_DATA_IN_LV: JP3.2, U1A.A2
- new net CP3_DATA_OUT_LV: JP5.4, JP8.4, U7G$1.A
- new net CP3_DATA_OUT_OE_LV: JP5.3, JP8.3, U7G$1.OE
- new net CP4_+3V3: C5.1, J9P4.2, JP1.1, U8G$2.VCC
- new net CP4_DATA: J9P4.3, JP2.2, U1A.B1, U8G$1.Y
- new net CP4_DATA_IN_LV: JP3.1, U1A.A1
- new net CP4_DATA_OUT_LV: JP5.2, JP8.2, U8G$1.A
- new net CP4_DATA_OUT_OE_LV: JP5.1, JP8.1, U8G$1.OE
- net +3V3: now also JP1.2, JP10.3; no longer J5.2, J6.2, J7.2, J8.2
- net DEBUG0: now also JP13.4, JP14.4; no longer JP6.1, JP9.1
- net DEBUG1: now also JP13.3, JP14.3; no longer JP6.2, JP9.2
- net DEBUG2: now also JP13.2, JP14.2; no longer JP6.3, JP9.3
- net DEBUG3: now also JP13.1, JP14.1; no longer JP6.4, JP9.4
- net DEBUG4: now also JP11.4, JP6.4; no longer JP6.5, JP9.5
- net DEBUG5: now also JP11.3, JP6.3; no longer JP6.6, JP9.6
- net DEBUG6: now also JP11.2, JP6.2; no longer JP6.7, JP9.7
- net DEBUG7: now also JP11.1, JP6.1; no longer JP6.8, JP9.8
- net GND: now also JP10.1, JP2.1, U1A.B5, U1A.B6, U1A.B7, U1A.B8; no longer J5.1, J6.1, J7.1, J8.1, JP1.1, JP13.1, JP21.1, U10G$2.GND, U3G$2.GND, U5G$2.GND, U9G$2.GND
Other:
- moved on the sheet: C1, J9P1, J9P2, J9P3, J9P4, J9SHLD, JP11, JP12, JP13, JP4, JP7, JP8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

Commit message: N64 PCB: Added controller ports with switches and mostly routed the board.
Parts:
- added C6, C7, C8, C9: 0.1u, rcl:C-EUC0603
- added J1: RJ45-S-4, TASLink:RJ45-S-4
- added JP15, JP16, JP17, JP19, JP20, JP21, JP22, JP23, JP24, JP9: (no value), SparkFun-Connectors:M04PTH
- added R1, R2, R3, R4: (no value), rcl:R-US_0207/2V
- added S1, S2, S3, S4, S5, S6, S7, S8: DPDT, TASLink:DPDT
- added U3, U5, U6, U9: MC74VHC1GT125, TASLink:MC74VHC1GT125
- JP1: value M02PTH -> (none); device SparkFun-Connectors:M02PTH -> SparkFun-Connectors:M04PTH
Connections:
- new net CP1_DIS_SIGNAL: JP3.1, R1.1, S1G$2.2
- new net CP2_DIS_SIGNAL: JP3.2, R2.1, S3G$2.2
- new net CP3_DIS_SIGNAL: JP3.3, R3.1, S5G$2.2
- new net CP4_DIS_SIGNAL: JP3.4, R4.1, S7G$2.2
- new net CTP1_+3V3: C6.1, J1P4.2, S2G$1.2, S2G$2.2, U3G$2.VCC
- new net CTP1_DATA: J1P4.3, JP20.1, S1G$1.1, U1A.B4, U3G$1.Y
- new net CTP1_DATA_IN_LV: JP11.4, U1A.A4
- new net CTP1_DATA_OUT_LV: JP1.3, JP22.3, U3G$1.A
- new net CTP1_DATA_OUT_OE_LV: JP1.4, JP22.4, U3G$1.OE
- new net CTP2_+3V3: C7.1, J1P3.2, S4G$1.2, S4G$2.2, U5G$2.VCC
- new net CTP2_DATA: J1P3.3, JP20.2, S3G$1.1, U1A.B3, U5G$1.Y
- new net CTP2_DATA_IN_LV: JP11.3, U1A.A3
- new net CTP2_DATA_OUT_LV: JP1.1, JP22.1, U5G$1.A
- new net CTP2_DATA_OUT_OE_LV: JP1.2, JP22.2, U5G$1.OE
- new net CTP3_+3V3: C8.1, J1P2.2, S6G$1.2, S6G$2.2, U6G$2.VCC
- new net CTP3_DATA: J1P2.3, JP20.3, S5G$1.1, U1A.B2, U6G$1.Y
- new net CTP3_DATA_IN_LV: JP11.2, U1A.A2
- new net CTP3_DATA_OUT_LV: JP23.2, JP9.2, U6G$1.A
- new net CTP3_DATA_OUT_OE_LV: JP23.1, JP9.1, U6G$1.OE
- new net CTP4_+3V3: C9.1, J1P1.2, S8G$1.2, S8G$2.2, U9G$2.VCC
- new net CTP4_DATA: J1P1.3, JP20.4, S7G$1.1, U1A.B1, U9G$1.Y
- new net CTP4_DATA_IN_LV: JP11.1, U1A.A1
- new net CTP4_DATA_OUT_LV: JP23.4, JP9.4, U9G$1.A
- new net CTP4_DATA_OUT_OE_LV: JP23.3, JP9.3, U9G$1.OE
- new net VP1_CLOCK: JP15.1
- new net VP1_D0: JP16.1
- new net VP1_D1: JP16.2
- new net VP1_D2: JP16.3
- new net VP1_D3: JP16.4
- new net VP1_LATCH: JP15.2
- net +3V3: now also JP24.3, R1.2, R2.2, R3.2, R4.2, S2G$1.3, S2G$2.3, S4G$1.3, S4G$2.3, S6G$1.3, S6G$2.3, S8G$1.3, S8G$2.3; no longer JP1.2, JP10.3
- net CP1_+3V3: now also S2G$1.1, S2G$2.1
- net CP1_DATA: now also JP2.2, S1G$1.2, U1A.B8; no longer JP2.5, U1A.B4
- net CP1_DATA_IN_LV: now also JP17.4, U1A.A8; no longer JP3.4, U1A.A4
- net CP2_+3V3: now also S4G$1.1, S4G$2.1
- net CP2_DATA: now also JP2.3, S3G$1.2, U1A.B7; no longer JP2.4, U1A.B3
- net CP2_DATA_IN_LV: now also JP17.3, U1A.A7; no longer JP3.3, U1A.A3
- net CP3_+3V3: now also S6G$1.1, S6G$2.1
- net CP3_DATA: now also JP2.4, S5G$1.2, U1A.B6; no longer JP2.3, U1A.B2
- net CP3_DATA_IN_LV: now also JP17.2, U1A.A6; no longer JP3.2, U1A.A2
- net CP4_+3V3: now also S8G$1.1, S8G$2.1; no longer JP1.1
- net CP4_DATA: now also JP2.5, S7G$1.2, U1A.B5; no longer JP2.2, U1A.B1
- net CP4_DATA_IN_LV: now also JP17.1, U1A.A5; no longer JP3.1, U1A.A1
- net DEBUG4: now also JP19.4; no longer JP11.4
- net DEBUG5: now also JP19.3; no longer JP11.3
- net DEBUG6: now also JP19.2; no longer JP11.2
- net DEBUG7: now also JP19.1; no longer JP11.1
- net GND: now also C6.2, C7.2, C8.2, C9.2, J1P1.1, J1P2.1, J1P3.1, J1P4.1, J1SHLD.S1, J1SHLD.S2, J1SHLD.S3, J1SHLD.S4, JP21.1, JP24.1, S1G$2.1, S3G$2.1, S5G$2.1, S7G$2.1, U3G$2.GND, U5G$2.GND, U6G$2.GND, U9G$2.GND; no longer U1A.B5, U1A.B6, U1A.B7, U1A.B8
Other:
- moved on the sheet: JP10, JP11, JP14, JP3, JP4, JP5

Commit message: N64 PCB: Added switches, controller ports, and many other features. Layout and routing mostly complete.
Parts:
- removed JP20: (no value), SparkFun-Connectors:M04PTH
- added JP18: M09, SparkFun-Connectors:M09
- JP2: device SparkFun-Connectors:M05PTH -> SparkFun-Connectors:M04PTH
Connections:
- net CP1_DATA: now also JP18.2; no longer JP2.2
- net CP2_DATA: now also JP18.3; no longer JP2.3
- net CP3_DATA: now also JP18.4; no longer JP2.4
- net CP4_DATA: now also JP18.5; no longer JP2.5
- net CTP1_DATA: now also JP18.6; no longer JP20.1
- net CTP2_DATA: now also JP18.7; no longer JP20.2
- net CTP3_DATA: now also JP18.8; no longer JP20.3
- net CTP4_DATA: now also JP18.9; no longer JP20.4
- net GND: now also JP18.1, JP2.2, JP2.3, JP2.4
